File: Camera.kicad_sch (KiCad schematic)
At the start: 25 parts, among them J11 camera, U10 RT9193-28GB, U8 RT9193-18GB, U9 RT9193-15GB

Commit message: hardware: update design and tapeout for fabrication
Parts:
- C31, C32, C33, C37, C38, C39: footprint Capacitor_SMD:C_0603_1608Metric -> RM_Guided_Dart_Base_HW-Footprints:C_0603_1608Metric; symbol Device:C_Small -> RM_Guided_Dart_Base_HW:C_Small
- C34, C35, C36, C40, C41, C42: footprint Capacitor_SMD:C_0402_1005Metric -> RM_Guided_Dart_Base_HW-Footprints:C_0402_1005Metric; symbol Device:C_Small -> RM_Guided_Dart_Base_HW:C_Small
- C43: footprint Capacitor_SMD:C_0603_1608Metric -> RM_Guided_Dart_Base_HW-Footprints:C_0603_1608Metric; symbol Device:C -> RM_Guided_Dart_Base_HW:C
- C44: footprint Capacitor_SMD:C_0402_1005Metric -> RM_Guided_Dart_Base_HW-Footprints:C_0402_1005Metric; symbol Device:C -> RM_Guided_Dart_Base_HW:C
- J11: footprint RWN_Footprints:FH12-24S-0.5SH_1x24-1MP_P0.50mm_Horizontal -> RM_Guided_Dart_Base_HW-Footprints:FH12-24S-0.5SH_1x24-1MP_P0.50mm_Horizontal; symbol Connector_Generic_MountingPin:Conn_01x24_MountingPin -> RM_Guided_Dart_Base_HW:Conn_01x24_MountingPin
- R32, R33, R34: footprint Resistor_SMD:R_0402_1005Metric -> RM_Guided_Dart_Base_HW-Footprints:R_0402_1005Metric; symbol Device:R_Small -> RM_Guided_Dart_Base_HW:R_Small
- R35, R36, R37, R38: footprint Resistor_SMD:R_0402_1005Metric -> RM_Guided_Dart_Base_HW-Footprints:R_0402_1005Metric; symbol Device:R -> RM_Guided_Dart_Base_HW:R
- U10, U8, U9: footprint Package_TO_SOT_SMD:SOT-23-5 -> RM_Guided_Dart_Base_HW-Footprints:SOT-23-5; symbol RWN_Symbols:RT9193 -> RM_Guided_Dart_Base_HW:RT9193_1
Changed lines of the file:
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@@
 	)
 	(symbol
-		(lib_id "Device:C_Small")
+		(lib_id "RM_Guided_Dart_Base_HW:C_Small")
 		(at 34.29 63.5 0)
 		(mirror y)
@@
 			)
 		)
-		(property "Footprint" "Capacitor_SMD:C_0603_1608Metric"
+		(property "Footprint" "RM_Guided_Dart_Base_HW-Footprints:C_0603_1608Metric"
 			(at 34.29 63.5 0)
 			(hide yes)
@@
 	)
 	(symbol
-		(lib_id "Device:C_Small")
+		(lib_id "RM_Guided_Dart_Base_HW:C_Small")
 		(at 69.85 38.1 0)
 		(mirror x)
@@
 			)
 		)
-		(property "Footprint" "Capacitor_SMD:C_0402_1005Metric"
+		(property "Footprint" "RM_Guided_Dart_Base_HW-Footprints:C_0402_1005Metric"
 			(at 69.85 38.1 0)
 			(hide yes)
@@
 	)
 	(symbol
-		(lib_id "Device:C")
+		(lib_id "RM_Guided_Dart_Base_HW:C")
 		(at 163.83 45.72 0)
 		(unit 1)
@@
 			)
 		)
-		(property "Footprint" "Capacitor_SMD:C_0402_1005Metric"
+		(property "Footprint" "RM_Guided_Dart_Base_HW-Footprints:C_0402_1005Metric"
 			(at 164.7952 49.53 0)
 			(hide yes)
@@
 	)
 	(symbol
-		(lib_id "Device:C_Small")
+		(lib_id "RM_Guided_Dart_Base_HW:C_Small")
 		(at 60.96 68.58 0)
 		(mirror x)
@@
 			)
 		)
-		(property "Footprint" "Capacitor_SMD:C_0603_1608Metric"
+		(property "Footprint" "RM_Guided_Dart_Base_HW-Footprints:C_0603_1608Metric"
 			(at 60.96 68.58 0)
 			(hide yes)
@@
 	(symbol
 		(lib_name "RT9193_1")
-		(lib_id "RWN_Symbols:RT9193")
+		(lib_id "RM_Guided_Dart_Base_HW:RT9193_1")
 		(at 44.45 35.56 0)
 		(unit 1)
@@
 			)
 		)
-		(property "Footprint" "Package_TO_SOT_SMD:SOT-23-5"
+		(property "Footprint" "RM_Guided_Dart_Base_HW-Footprints:SOT-23-5"
 			(at 44.45 35.56 0)
 			(hide yes)
@@
 	)
 	(symbol
-		(lib_id "Device:R")
+		(lib_id "RM_Guided_Dart_Base_HW:R")
 		(at 161.29 78.74 0)
 		(unit 1)
@@
 			)
 		)
-		(property "Footprint" "Resistor_SMD:R_0402_1005Metric"
+		(property "Footprint" "RM_Guided_Dart_Base_HW-Footprints:R_0402_1005Metric"
 			(at 159.512 78.74 90)
 			(hide yes)
@@
 	)
 	(symbol
-		(lib_id "Device:R_Small")
+		(lib_id "RM_Guided_Dart_Base_HW:R_Small")
 		(at 26.67 66.04 180)
 		(unit 1)
@@
 			)
 		)
-		(property "Footprint" "Resistor_SMD:R_0402_1005Metric"
+		(property "Footprint" "RM_Guided_Dart_Base_HW-Footprints:R_0402_1005Metric"
 			(at 26.67 66.04 0)
 			(hide yes)
@@
 	)
 	(symbol
-		(lib_id "Device:R_Small")
+		(lib_id "RM_Guided_Dart_Base_HW:R_Small")
 		(at 26.67 96.52 180)
 		(unit 1)
@@
 			)
 		)
-		(property "Footprint" "Resistor_SMD:R_0402_1005Metric"
+		(property "Footprint" "RM_Guided_Dart_Base_HW-Footprints:R_0402_1005Metric"
 			(at 26.67 96.52 0)
 			(hide yes)
@@
 	)
 	(symbol
-		(lib_id "Device:R")
+		(lib_id "RM_Guided_Dart_Base_HW:R")
 		(at 149.86 78.74 0)
 		(unit 1)
@@
 			)
 		)
-		(property "Footprint" "Resistor_SMD:R_0402_1005Metric"
+		(property "Footprint" "RM_Guided_Dart_Base_HW-Footprints:R_0402_1005Metric"
 			(at 148.082 78.74 90)
 			(hide yes)
@@
 	)
 	(symbol
-		(lib_id "Device:C_Small")
+		(lib_id "RM_Guided_Dart_Base_HW:C_Small")
 		(at 53.34 41.91 0)
 		(mirror x)
@@
 			)
 		)
-		(property "Footprint" "Capacitor_SMD:C_0402_1005Metric"
+		(property "Footprint" "RM_Guided_Dart_Base_HW-Footprints:C_0402_1005Metric"
 			(at 53.34 41.91 0)
 			(hide yes)
@@
 	)
 	(symbol
-		(lib_id "Device:C_Small")
+		(lib_id "RM_Guided_Dart_Base_HW:C_Small")
 		(at 34.29 33.02 0)
 		(mirror y)
@@
 			)
 		)
-		(property "Footprint" "Capacitor_SMD:C_0603_1608Metric"
+		(property "Footprint" "RM_Guided_Dart_Base_HW-Footprints:C_0603_1608Metric"
 			(at 34.29 33.02 0)
 			(hide yes)
@@
 	)
 	(symbol
-		(lib_id "Device:C_Small")
+		(lib_id "RM_Guided_Dart_Base_HW:C_Small")
 		(at 53.34 72.39 0)
 		(mirror x)
@@
 			)
 		)
-		(property "Footprint" "Capacitor_SMD:C_0402_1005Metric"
+		(property "Footprint" "RM_Guided_Dart_Base_HW-Footprints:C_0402_1005Metric"
 			(at 53.34 72.39 0)
 			(hide yes)
@@
 	)
 	(symbol
-		(lib_id "Device:C_Small")
+		(lib_id "RM_Guided_Dart_Base_HW:C_Small")
 		(at 53.34 102.87 0)
 		(mirror x)
@@
 			)
 		)
-		(property "Footprint" "Capacitor_SMD:C_0402_1005Metric"
+		(property "Footprint" "RM_Guided_Dart_Base_HW-Footprints:C_0402_1005Metric"
 			(at 53.34 102.87 0)
 			(hide yes)
@@
 	)
 	(symbol
-		(lib_id "Device:R_Small")
+		(lib_id "RM_Guided_Dart_Base_HW:R_Small")
 		(at 26.67 35.56 180)
 		(unit 1)
@@
 			)
 		)
-		(property "Footprint" "Resistor_SMD:R_0402_1005Metric"
+		(property "Footprint" "RM_Guided_Dart_Base_HW-Footprints:R_0402_1005Metric"
 			(at 26.67 35.56 0)
 			(hide yes)
@@
 	)
 	(symbol
-		(lib_id "Device:R")
+		(lib_id "RM_Guided_Dart_Base_HW:R")
 		(at 172.72 78.74 0)
 		(unit 1)
@@
 			)
 		)
-		(property "Footprint" "Resistor_SMD:R_0402_1005Metric"
+		(property "Footprint" "RM_Guided_Dart_Base_HW-Footprints:R_0402_1005Metric"
 			(at 170.942 78.74 90)
 			(hide yes)
@@
 	)
 	(symbol
-		(lib_id "Device:R")
+		(lib_id "RM_Guided_Dart_Base_HW:R")
 		(at 184.15 78.74 0)
 		(unit 1)
@@
 			)
 		)
-		(property "Footprint" "Resistor_SMD:R_0402_1005Metric"
+		(property "Footprint" "RM_Guided_Dart_Base_HW-Footprints:R_0402_1005Metric"
 			(at 182.372 78.74 90)
 			(hide yes)
@@
 	)
 	(symbol
-		(lib_id "Device:C_Small")
+		(lib_id "RM_Guided_Dart_Base_HW:C_Small")
 		(at 69.85 68.58 0)
 		(mirror x)
@@
 			)
 		)
-		(property "Footprint" "Capacitor_SMD:C_0402_1005Metric"
+		(property "Footprint" "RM_Guided_Dart_Base_HW-Footprints:C_0402_1005Metric"
 			(at 69.85 68.58 0)
 			(hide yes)
@@
 	)
 	(symbol
-		(lib_id "Device:C_Small")
+		(lib_id "RM_Guided_Dart_Base_HW:C_Small")
 		(at 34.29 93.98 0)
 		(mirror y)
@@
 			)
 		)
-		(property "Footprint" "Capacitor_SMD:C_0603_1608Metric"
+		(property "Footprint" "RM_Guided_Dart_Base_HW-Footprints:C_0603_1608Metric"
 			(at 34.29 93.98 0)
 			(hide yes)
@@
 	)
 	(symbol
-		(lib_id "Device:C_Small")
+		(lib_id "RM_Guided_Dart_Base_HW:C_Small")
 		(at 60.96 99.06 0)
 		(mirror x)
@@
 			)
 		)
-		(property "Footprint" "Capacitor_SMD:C_0603_1608Metric"
+		(property "Footprint" "RM_Guided_Dart_Base_HW-Footprints:C_0603_1608Metric"
 			(at 60.96 99.06 0)
 			(hide yes)
@@
 	)
 	(symbol
-		(lib_id "Device:C_Small")
+		(lib_id "RM_Guided_Dart_Base_HW:C_Small")
 		(at 69.85 99.06 0)
 		(mirror x)
@@
 			)
 		)
-		(property "Footprint" "Capacitor_SMD:C_0402_1005Metric"
+		(property "Footprint" "RM_Guided_Dart_Base_HW-Footprints:C_0402_1005Metric"
 			(at 69.85 99.06 0)
 			(hide yes)
@@
 	(symbol
 		(lib_name "RT9193_1")
-		(lib_id "RWN_Symbols:RT9193")
+		(lib_id "RM_Guided_Dart_Base_HW:RT9193_1")
 		(at 44.45 96.52 0)
 		(unit 1)
@@
 			)
 		)
-		(property "Footprint" "Package_TO_SOT_SMD:SOT-23-5"
+		(property "Footprint" "RM_Guided_Dart_Base_HW-Footprints:SOT-23-5"
 			(at 44.45 96.52 0)
 			(hide yes)
@@
 	(symbol
 		(lib_name "RT9193_1")
-		(lib_id "RWN_Symbols:RT9193")
+		(lib_id "RM_Guided_Dart_Base_HW:RT9193_1")
 		(at 44.45 66.04 0)
 		(unit 1)
@@
 			)
 		)
-		(property "Footprint" "Package_TO_SOT_SMD:SOT-23-5"
+		(property "Footprint" "RM_Guided_Dart_Base_HW-Footprints:SOT-23-5"
 			(at 44.45 66.04 0)
 			(hide yes)
@@
 	)
 	(symbol
-		(lib_id "Device:C")
+		(lib_id "RM_Guided_Dart_Base_HW:C")
 		(at 151.13 45.72 0)
 		(unit 1)
@@
 			)
 		)
-		(property "Footprint" "Capacitor_SMD:C_0603_1608Metric"
+		(property "Footprint" "RM_Guided_Dart_Base_HW-Footprints:C_0603_1608Metric"
 			(at 152.0952 49.53 0)
 			(hide yes)
@@
 	)
 	(symbol
-		(lib_id "Connector_Generic_MountingPin:Conn_01x24_MountingPin")
+		(lib_id "RM_Guided_Dart_Base_HW:Conn_01x24_MountingPin")
 		(at 124.46 53.34 0)
 		(mirror y)
@@
 			)
 		)
-		(property "Footprint" "RWN_Footprints:FH12-24S-0.5SH_1x24-1MP_P0.50mm_Horizontal"
+		(property "Footprint" "RM_Guided_Dart_Base_HW-Footprints:FH12-24S-0.5SH_1x24-1MP_P0.50mm_Horizontal"
 			(at 124.46 53.34 0)
 			(hide yes)
@@
 	)
 	(symbol
-		(lib_id "Device:C_Small")
+		(lib_id "RM_Guided_Dart_Base_HW:C_Small")
 		(at 60.96 38.1 0)
 		(mirror x)
@@
 			)
 		)
-		(property "Footprint" "Capacitor_SMD:C_0603_1608Metric"
+		(property "Footprint" "RM_Guided_Dart_Base_HW-Footprints:C_0603_1608Metric"
 			(at 60.96 38.1 0)
 			(hide yes)

Commit message: V1.2已打板
Parts:
- renumbered C31 to C32, C32 to C33, C33 to C34, C34 to C35, C35 to C36, C36 to C37, C37 to C38, C38 to C39, C39 to C40, C40 to C41, C41 to C42, C42 to C43, C43 to C44, C44 to C45, J11 to J12, R32 to R35, R33 to R36, R34 to R37, R35 to R38, R36 to R39, R37 to R40, R38 to R41
