File: IMU.kicad_sch (KiCad schematic)
At the start: 5 parts, among them U11 BMI088

Commit message: hardware: update design and tapeout for fabrication
Parts:
- C45, C46: footprint Capacitor_SMD:C_0402_1005Metric -> RM_Guided_Dart_Base_HW-Footprints:C_0402_1005Metric; symbol Device:C -> RM_Guided_Dart_Base_HW:C
- R39: footprint Resistor_SMD:R_0603_1608Metric -> RM_Guided_Dart_Base_HW-Footprints:R_0603_1608Metric; symbol Library:R -> RM_Guided_Dart_Base_HW:R
- R40: footprint Resistor_SMD:R_0603_1608Metric -> RM_Guided_Dart_Base_HW-Footprints:R_0603_1608Metric; symbol Device:R -> RM_Guided_Dart_Base_HW:R
- U11: footprint Package_LGA:Bosch_LGA-16_4.5x3mm_P0.5mm_LayoutBorder7x1y_ClockwisePinNumbering -> RM_Guided_Dart_Base_HW-Footprints:Bosch_LGA-16_4.5x3mm_P0.5mm_LayoutBorder7x1y_ClockwisePinNumbering; symbol Library:BMI088 -> RM_Guided_Dart_Base_HW:BMI088
Connections:
- net GND: now also U11.2 (NC)
- no-connect marks 2 -> 1
Changed lines of the file:
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@@
+	)
+	(junction
+		(at 97.79 68.58)
+		(diameter 0)
+		(color 0 0 0 0)
 	)
 	(junction
@@
 	)
 	(no_connect
-		(at 95.25 68.58)
-	)
-	(no_connect
 		(at 95.25 60.96)
 	)
@@
 	(wire
 		(pts
-			(xy 97.79 76.2) (xy 97.79 66.04)
+			(xy 97.79 76.2) (xy 97.79 68.58)
 		)
 		(stroke
@@
 	(wire
 		(pts
+			(xy 97.79 68.58) (xy 97.79 66.04)
+		)
+		(stroke
+			(width 0)
+			(type default)
+		)
+	)
+	(wire
+		(pts
 			(xy 110.49 53.34) (xy 95.25 53.34)
 		)
@@
 		(pts
 			(xy 69.85 60.96) (xy 68.58 60.96)
+		)
+		(stroke
+			(width 0)
+			(type default)
+		)
+	)
+	(wire
+		(pts
+			(xy 95.25 68.58) (xy 97.79 68.58)
 		)
 		(stroke
@@
 	)
 	(symbol
-		(lib_id "Library:R")
+		(lib_id "RM_Guided_Dart_Base_HW:R")
 		(at 59.69 60.96 90)
 		(unit 1)
@@
 			)
 		)
-		(property "Footprint" "Resistor_SMD:R_0603_1608Metric"
+		(property "Footprint" "RM_Guided_Dart_Base_HW-Footprints:R_0603_1608Metric"
 			(at 59.69 62.738 90)
 			(hide yes)
@@
 	)
 	(symbol
-		(lib_id "Library:BMI088")
+		(lib_id "RM_Guided_Dart_Base_HW:BMI088")
 		(at 82.55 60.96 0)
 		(unit 1)
@@
 			)
 		)
-		(property "Footprint" "Package_LGA:Bosch_LGA-16_4.5x3mm_P0.5mm_LayoutBorder7x1y_ClockwisePinNumbering"
+		(property "Footprint" "RM_Guided_Dart_Base_HW-Footprints:Bosch_LGA-16_4.5x3mm_P0.5mm_LayoutBorder7x1y_ClockwisePinNumbering"
 			(at 82.55 60.96 0)
 			(hide yes)
@@
 	)
 	(symbol
-		(lib_id "Device:R")
+		(lib_id "RM_Guided_Dart_Base_HW:R")
 		(at 102.87 59.69 0)
 		(unit 1)
@@
 			)
 		)
-		(property "Footprint" "Resistor_SMD:R_0603_1608Metric"
+		(property "Footprint" "RM_Guided_Dart_Base_HW-Footprints:R_0603_1608Metric"
 			(at 101.092 59.69 90)
 			(hide yes)
@@
 	)
 	(symbol
-		(lib_id "Device:C")
+		(lib_id "RM_Guided_Dart_Base_HW:C")
 		(at 147.32 59.69 0)
 		(unit 1)
@@
 			)
 		)
-		(property "Footprint" "Capacitor_SMD:C_0402_1005Metric"
+		(property "Footprint" "RM_Guided_Dart_Base_HW-Footprints:C_0402_1005Metric"
 			(at 148.2852 63.5 0)
 			(hide yes)
@@
 	)
 	(symbol
-		(lib_id "Device:C")
+		(lib_id "RM_Guided_Dart_Base_HW:C")
 		(at 137.16 59.69 0)
 		(unit 1)
@@
 			)
 		)
-		(property "Footprint" "Capacitor_SMD:C_0402_1005Metric"
+		(property "Footprint" "RM_Guided_Dart_Base_HW-Footprints:C_0402_1005Metric"
 			(at 138.1252 63.5 0)
 			(hide yes)

Commit message: V1.2已打板
Parts:
- renumbered C45 to C46, C46 to C47, R39 to R42, R40 to R43
Changed lines of the file:
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@@
 		(dnp no)
 		(fields_autoplaced yes)
-		(property "Reference" "#PWR0105"
+		(property "Reference" "#PWR0115"
 			(at 97.79 82.55 0)
 			(hide yes)
@@
 			(project "RM_Guided_Dart_Base_HW"
 				(path "/6ed09268-0e95-41b2-b676-0d7bbc40f5ee/8622f810-d5b7-4ecf-9f23-e3bd128862ca"
-					(reference "#PWR0105")
+					(reference "#PWR0115")
 					(unit 1)
 				)
@@
 		(in_pos_files yes)
 		(dnp no)
-		(property "Reference" "R39"
+		(property "Reference" "R42"
 			(at 57.15 63.246 90)
 			(show_name no)
@@
 			(project "RM_Guided_Dart_Base_HW"
 				(path "/6ed09268-0e95-41b2-b676-0d7bbc40f5ee/8622f810-d5b7-4ecf-9f23-e3bd128862ca"
-					(reference "R39")
+					(reference "R42")
 					(unit 1)
 				)
@@
 		(dnp no)
 		(fields_autoplaced yes)
-		(property "Reference" "#PWR0104"
+		(property "Reference" "#PWR0114"
 			(at 82.55 82.55 0)
 			(hide yes)
@@
 			(project "RM_Guided_Dart_Base_HW"
 				(path "/6ed09268-0e95-41b2-b676-0d7bbc40f5ee/8622f810-d5b7-4ecf-9f23-e3bd128862ca"
-					(reference "#PWR0104")
+					(reference "#PWR0114")
 					(unit 1)
 				)
@@
 		(dnp no)
 		(fields_autoplaced yes)
-		(property "Reference" "#PWR0107"
+		(property "Reference" "#PWR0117"
 			(at 137.16 81.28 0)
 			(hide yes)
@@
 			(project "RM_Guided_Dart_Base_HW"
 				(path "/6ed09268-0e95-41b2-b676-0d7bbc40f5ee/8622f810-d5b7-4ecf-9f23-e3bd128862ca"
-					(reference "#PWR0107")
+					(reference "#PWR0117")
 					(unit 1)
 				)
@@
 		(dnp no)
 		(fields_autoplaced yes)
-		(property "Reference" "R40"
+		(property "Reference" "R43"
 			(at 105.41 58.4199 0)
 			(show_name no)
@@
 			(project "RM_Guided_Dart_Base_HW"
 				(path "/6ed09268-0e95-41b2-b676-0d7bbc40f5ee/8622f810-d5b7-4ecf-9f23-e3bd128862ca"
-					(reference "R40")
+					(reference "R43")
 					(unit 1)
 				)
@@
 		(dnp no)
 		(fields_autoplaced yes)
-		(property "Reference" "#PWR0108"
+		(property "Reference" "#PWR0118"
 			(at 147.32 48.26 0)
 			(hide yes)
@@
 			(project "RM_Guided_Dart_Base_HW"
 				(path "/6ed09268-0e95-41b2-b676-0d7bbc40f5ee/8622f810-d5b7-4ecf-9f23-e3bd128862ca"
-					(reference "#PWR0108")
+					(reference "#PWR0118")
 					(unit 1)
 				)
@@
 		(dnp no)
 		(fields_autoplaced yes)
-		(property "Reference" "#PWR0106"
+		(property "Reference" "#PWR0116"
 			(at 137.16 48.26 0)
 			(hide yes)
@@
 			(project "RM_Guided_Dart_Base_HW"
 				(path "/6ed09268-0e95-41b2-b676-0d7bbc40f5ee/8622f810-d5b7-4ecf-9f23-e3bd128862ca"
-					(reference "#PWR0106")
+					(reference "#PWR0116")
 					(unit 1)
 				)
@@
 		(in_pos_files yes)
 		(dnp no)
-		(property "Reference" "C46"
+		(property "Reference" "C47"
 			(at 149.606 58.42 0)
 			(show_name no)
@@
 			(project "RM_Guided_Dart_Base_HW"
 				(path "/6ed09268-0e95-41b2-b676-0d7bbc40f5ee/8622f810-d5b7-4ecf-9f23-e3bd128862ca"
-					(reference "C46")
+					(reference "C47")
 					(unit 1)
 				)
@@
 		(dnp no)
 		(fields_autoplaced yes)
-		(property "Reference" "#PWR0103"
+		(property "Reference" "#PWR0113"
 			(at 82.55 49.53 0)
 			(hide yes)
@@
 			(project "RM_Guided_Dart_Base_HW"
 				(path "/6ed09268-0e95-41b2-b676-0d7bbc40f5ee/8622f810-d5b7-4ecf-9f23-e3bd128862ca"
-					(reference "#PWR0103")
+					(reference "#PWR0113")
 					(unit 1)
 				)
@@
 		(dnp no)
 		(fields_autoplaced yes)
-		(property "Reference" "#PWR0109"
+		(property "Reference" "#PWR0119"
 			(at 147.32 81.28 0)
 			(hide yes)
@@
 			(project "RM_Guided_Dart_Base_HW"
 				(path "/6ed09268-0e95-41b2-b676-0d7bbc40f5ee/8622f810-d5b7-4ecf-9f23-e3bd128862ca"
-					(reference "#PWR0109")
+					(reference "#PWR0119")
 					(unit 1)
 				)
@@
 		(in_pos_files yes)
 		(dnp no)
-		(property "Reference" "C45"
+		(property "Reference" "C46"
 			(at 139.446 58.42 0)
 			(show_name no)
@@
 			(project "RM_Guided_Dart_Base_HW"
 				(path "/6ed09268-0e95-41b2-b676-0d7bbc40f5ee/8622f810-d5b7-4ecf-9f23-e3bd128862ca"
-					(reference "C45")
-					(unit 1)
-				)
+					(reference "C46")
+					(unit 1)
+				)
