File: Power.kicad_sch (KiCad schematic)
At the start: 20 parts, among them U3 SY8303AIC, U4 SY8303AIC

Commit message: hardware: update design and tapeout for fabrication
Parts:
- C1, C10, C2, C9: footprint Capacitor_SMD:C_0603_1608Metric -> RM_Guided_Dart_Base_HW-Footprints:C_0603_1608Metric; symbol library:C -> RM_Guided_Dart_Base_HW:C
- C3, C4, C5, C6, C7, C8: footprint Capacitor_SMD:C_0402_1005Metric -> RM_Guided_Dart_Base_HW-Footprints:C_0402_1005Metric; symbol library:C -> RM_Guided_Dart_Base_HW:C
- L1, L2: footprint Inductor_SMD:L_Changjiang_FTC303020D -> RM_Guided_Dart_Base_HW-Footprints:L_Changjiang_FTC303020D; symbol library:L -> RM_Guided_Dart_Base_HW:L
- R10, R11, R12, R13, R8, R9: footprint Resistor_SMD:R_0402_1005Metric -> RM_Guided_Dart_Base_HW-Footprints:R_0402_1005Metric; symbol library:R -> RM_Guided_Dart_Base_HW:R
- U3, U4: footprint Package_TO_SOT_SMD:TSOT-23-8 -> RM_Guided_Dart_Base_HW-Footprints:TSOT-23-8; symbol library:SY8303AIC -> RM_Guided_Dart_Base_HW:SY8303AIC
Changed lines of the file:
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@@
 	)
 	(symbol
-		(lib_id "library:C")
+		(lib_id "RM_Guided_Dart_Base_HW:C")
 		(at 73.66 26.67 0)
 		(unit 1)
@@
 			)
 		)
-		(property "Footprint" "Capacitor_SMD:C_0402_1005Metric"
+		(property "Footprint" "RM_Guided_Dart_Base_HW-Footprints:C_0402_1005Metric"
 			(at 74.6252 30.48 0)
 			(hide yes)
@@
 	)
 	(symbol
-		(lib_id "library:C")
+		(lib_id "RM_Guided_Dart_Base_HW:C")
 		(at 111.76 87.63 0)
 		(unit 1)
@@
 			)
 		)
-		(property "Footprint" "Capacitor_SMD:C_0603_1608Metric"
+		(property "Footprint" "RM_Guided_Dart_Base_HW-Footprints:C_0603_1608Metric"
 			(at 112.7252 91.44 0)
 			(hide yes)
@@
 	)
 	(symbol
-		(lib_id "library:C")
+		(lib_id "RM_Guided_Dart_Base_HW:C")
 		(at 27.94 78.74 0)
 		(unit 1)
@@
 			)
 		)
-		(property "Footprint" "Capacitor_SMD:C_0603_1608Metric"
+		(property "Footprint" "RM_Guided_Dart_Base_HW-Footprints:C_0603_1608Metric"
 			(at 28.9052 82.55 0)
 			(hide yes)
@@
 	)
 	(symbol
-		(lib_id "library:SY8303AIC")
+		(lib_id "RM_Guided_Dart_Base_HW:SY8303AIC")
 		(at 59.69 77.47 0)
 		(unit 1)
@@
 			)
 		)
-		(property "Footprint" "Package_TO_SOT_SMD:TSOT-23-8"
+		(property "Footprint" "RM_Guided_Dart_Base_HW-Footprints:TSOT-23-8"
 			(at 59.69 77.47 0)
 			(hide yes)
@@
 	)
 	(symbol
-		(lib_id "library:C")
+		(lib_id "RM_Guided_Dart_Base_HW:C")
 		(at 73.66 72.39 0)
 		(unit 1)
@@
 			)
 		)
-		(property "Footprint" "Capacitor_SMD:C_0402_1005Metric"
+		(property "Footprint" "RM_Guided_Dart_Base_HW-Footprints:C_0402_1005Metric"
 			(at 74.6252 76.2 0)
 			(hide yes)
@@
 	)
 	(symbol
-		(lib_id "library:C")
+		(lib_id "RM_Guided_Dart_Base_HW:C")
 		(at 27.94 33.02 0)
 		(unit 1)
@@
 			)
 		)
-		(property "Footprint" "Capacitor_SMD:C_0603_1608Metric"
+		(property "Footprint" "RM_Guided_Dart_Base_HW-Footprints:C_0603_1608Metric"
 			(at 28.9052 36.83 0)
 			(hide yes)
@@
 	)
 	(symbol
-		(lib_id "library:L")
+		(lib_id "RM_Guided_Dart_Base_HW:L")
 		(at 78.74 77.47 90)
 		(unit 1)
@@
 			)
 		)
-		(property "Footprint" "Inductor_SMD:L_Changjiang_FTC303020D"
+		(property "Footprint" "RM_Guided_Dart_Base_HW-Footprints:L_Changjiang_FTC303020D"
 			(at 78.74 77.47 0)
 			(hide yes)
@@
 	)
 	(symbol
-		(lib_id "library:C")
+		(lib_id "RM_Guided_Dart_Base_HW:C")
 		(at 86.36 36.83 0)
 		(unit 1)
@@
 			)
 		)
-		(property "Footprint" "Capacitor_SMD:C_0402_1005Metric"
+		(property "Footprint" "RM_Guided_Dart_Base_HW-Footprints:C_0402_1005Metric"
 			(at 87.3252 40.64 0)
 			(hide yes)
@@
 	)
 	(symbol
-		(lib_id "library:L")
+		(lib_id "RM_Guided_Dart_Base_HW:L")
 		(at 78.74 31.75 90)
 		(unit 1)
@@
 			)
 		)
-		(property "Footprint" "Inductor_SMD:L_Changjiang_FTC303020D"
+		(property "Footprint" "RM_Guided_Dart_Base_HW-Footprints:L_Changjiang_FTC303020D"
 			(at 78.74 31.75 0)
 			(hide yes)
@@
 	)
 	(symbol
-		(lib_id "library:C")
+		(lib_id "RM_Guided_Dart_Base_HW:C")
 		(at 39.37 33.02 0)
 		(unit 1)
@@
 			)
 		)
-		(property "Footprint" "Capacitor_SMD:C_0402_1005Metric"
+		(property "Footprint" "RM_Guided_Dart_Base_HW-Footprints:C_0402_1005Metric"
 			(at 40.3352 36.83 0)
 			(hide yes)
@@
 	)
 	(symbol
-		(lib_id "library:C")
+		(lib_id "RM_Guided_Dart_Base_HW:C")
 		(at 111.76 41.91 0)
 		(unit 1)
@@
 			)
 		)
-		(property "Footprint" "Capacitor_SMD:C_0603_1608Metric"
+		(property "Footprint" "RM_Guided_Dart_Base_HW-Footprints:C_0603_1608Metric"
 			(at 112.7252 45.72 0)
 			(hide yes)
@@
 	)
 	(symbol
-		(lib_id "library:SY8303AIC")
+		(lib_id "RM_Guided_Dart_Base_HW:SY8303AIC")
 		(at 59.69 31.75 0)
 		(unit 1)
@@
 			)
 		)
-		(property "Footprint" "Package_TO_SOT_SMD:TSOT-23-8"
+		(property "Footprint" "RM_Guided_Dart_Base_HW-Footprints:TSOT-23-8"
 			(at 59.69 31.75 0)
 			(hide yes)
@@
 	)
 	(symbol
-		(lib_id "library:C")
+		(lib_id "RM_Guided_Dart_Base_HW:C")
 		(at 86.36 82.55 0)
 		(unit 1)
@@
 			)
 		)
-		(property "Footprint" "Capacitor_SMD:C_0402_1005Metric"
+		(property "Footprint" "RM_Guided_Dart_Base_HW-Footprints:C_0402_1005Metric"
 			(at 87.3252 86.36 0)
 			(hide yes)
@@
 	)
 	(symbol
-		(lib_id "library:R")
+		(lib_id "RM_Guided_Dart_Base_HW:R")
 		(at 41.91 91.44 180)
 		(unit 1)
@@
 			)
 		)
-		(property "Footprint" "Resistor_SMD:R_0402_1005Metric"
+		(property "Footprint" "RM_Guided_Dart_Base_HW-Footprints:R_0402_1005Metric"
 			(at 43.688 91.44 90)
 			(hide yes)
@@
 	)
 	(symbol
-		(lib_id "library:C")
+		(lib_id "RM_Guided_Dart_Base_HW:C")
 		(at 39.37 78.74 0)
 		(unit 1)
@@
 			)
 		)
-		(property "Footprint" "Capacitor_SMD:C_0402_1005Metric"
+		(property "Footprint" "RM_Guided_Dart_Base_HW-Footprints:C_0402_1005Metric"
 			(at 40.3352 82.55 0)
 			(hide yes)
@@
 	)
 	(symbol
-		(lib_id "library:R")
+		(lib_id "RM_Guided_Dart_Base_HW:R")
 		(at 96.52 36.83 180)
 		(unit 1)
@@
 			)
 		)
-		(property "Footprint" "Resistor_SMD:R_0402_1005Metric"
+		(property "Footprint" "RM_Guided_Dart_Base_HW-Footprints:R_0402_1005Metric"
 			(at 98.298 36.83 90)
 			(hide yes)
@@
 	)
 	(symbol
-		(lib_id "library:R")
+		(lib_id "RM_Guided_Dart_Base_HW:R")
 		(at 96.52 82.55 180)
 		(unit 1)
@@
 			)
 		)
-		(property "Footprint" "Resistor_SMD:R_0402_1005Metric"
+		(property "Footprint" "RM_Guided_Dart_Base_HW-Footprints:R_0402_1005Metric"
 			(at 98.298 82.55 90)
 			(hide yes)
@@
 	)
 	(symbol
-		(lib_id "library:R")
+		(lib_id "RM_Guided_Dart_Base_HW:R")
 		(at 96.52 46.99 180)
 		(unit 1)
@@
 			)
 		)
-		(property "Footprint" "Resistor_SMD:R_0402_1005Metric"
+		(property "Footprint" "RM_Guided_Dart_Base_HW-Footprints:R_0402_1005Metric"
 			(at 98.298 46.99 90)
 			(hide yes)
@@
 	)
 	(symbol
-		(lib_id "library:R")
+		(lib_id "RM_Guided_Dart_Base_HW:R")
 		(at 96.52 92.71 180)
 		(unit 1)
@@
 			)
 		)
-		(property "Footprint" "Resistor_SMD:R_0402_1005Metric"
+		(property "Footprint" "RM_Guided_Dart_Base_HW-Footprints:R_0402_1005Metric"
 			(at 98.298 92.71 90)
 			(hide yes)
@@
 	)
 	(symbol
-		(lib_id "library:R")
+		(lib_id "RM_Guided_Dart_Base_HW:R")
 		(at 41.91 46.99 180)
 		(unit 1)
@@
 			)
 		)
-		(property "Footprint" "Resistor_SMD:R_0402_1005Metric"
+		(property "Footprint" "RM_Guided_Dart_Base_HW-Footprints:R_0402_1005Metric"
 			(at 43.688 46.99 90)
 			(hide yes)
