File: RM_Guided_Dart_Base_HW.kicad_pcb (KiCad board)
At the start: 4 copper layers, 80 x 32 mm, 129 parts, among them J1 CSI, J10 Battery, J11 camera, J2 DSI, J3 JTAG, J4 UART3, J5 PWM1, J6 PWM2, J7 PWM3, J8 PWM4, J9 USB_C_Receptacle_USB2.0_14P, Q1 AON7544, Q2 AON7544, SW1 SW_Push, SW2 SW_Push_DPDT, U1 LicheeRV_Nano, U10 RT9193-28GB, U11 BMI088, U2 XIAO-ESP32-C5-DIP, U3 SY8303AIC, U4 SY8303AIC, U5 CH224Q, U6 TP5100, U7 TPS54620RHLR, U8 RT9193-18GB, U9 RT9193-15GB

Commit message: hardware: update design and tapeout for fabrication
Parts:
- added G***: LOGO, LOGO, F.Cu at (117.3, 109.1)
- added G***: LOGO, LOGO, F.Cu at (100.8, 96.0)
- added G***: LOGO, LOGO, F.Cu at (105.9, 109.2)
- C1, C10, C11, C13, C14, C15, C2, C22, C23, C31, C32, C33, C37, C38, C39, C43, C9: footprint Capacitor_SMD:C_0603_1608Metric -> RM_Guided_Dart_Base_HW-Footprints:C_0603_1608Metric
- C12, C16, C17, C18, C19, C20, C21, C24, C25, C26, C3, C30, C34, C35, C36, C4, C40, C41, C42, C44, C45, C46, C5, C6, C7, C8: footprint Capacitor_SMD:C_0402_1005Metric -> RM_Guided_Dart_Base_HW-Footprints:C_0402_1005Metric
- C27, C28: value 47uF -> 22uF; footprint Capacitor_SMD:C_0603_1608Metric -> RM_Guided_Dart_Base_HW-Footprints:C_0603_1608Metric
- C29, C47: footprint Capacitor_SMD:C_1206_3216Metric -> RM_Guided_Dart_Base_HW-Footprints:C_1206_3216Metric
- D1, D2, D3, D4, D5: footprint LED_SMD:LED_0402_1005Metric -> RM_Guided_Dart_Base_HW-Footprints:LED_0402_1005Metric
- D6, D7: footprint Diode_SMD:D_SMA -> RM_Guided_Dart_Base_HW-Footprints:D_SMA
- D8: footprint Diode_SMD:D_SOD-323 -> RM_Guided_Dart_Base_HW-Footprints:D_SOD-323
- H1, H2, H3, H4: footprint MountingHole:MountingHole_3.2mm_M3_Pad_Via -> RM_Guided_Dart_Base_HW-Footprints:MountingHole_3.2mm_M3_Pad_Via
- J1: footprint RWN_Footprints:FPC-SMD_22P-P1.00_AFC11-S22ICC-00 -> RM_Guided_Dart_Base_HW-Footprints:FPC-SMD_22P-P1.00_AFC11-S22ICC-00
- J10: footprint RWN_Footprints:AMASS_XT30APW-M_1x02_P2.50mm_Horizontal -> RM_Guided_Dart_Base_HW-Footprints:AMASS_XT30APW-M_1x02_P2.50mm_Horizontal
- J11: footprint RWN_Footprints:FH12-24S-0.5SH_1x24-1MP_P0.50mm_Horizontal -> RM_Guided_Dart_Base_HW-Footprints:FH12-24S-0.5SH_1x24-1MP_P0.50mm_Horizontal
- J2: footprint Connector_FFC-FPC:Hirose_FH26-31S-0.3SHW_2Rows-31Pins-1MP_P0.60mm_Horizontal -> RM_Guided_Dart_Base_HW-Footprints:Hirose_FH26-31S-0.3SHW_2Rows-31Pins-1MP_P0.60mm_Horizontal
- J3: footprint Connector_JST:JST_GH_SM06B-GHS-TB_1x06-1MP_P1.25mm_Horizontal -> RM_Guided_Dart_Base_HW-Footprints:JST_GH_SM06B-GHS-TB_1x06-1MP_P1.25mm_Horizontal
- J4: footprint Connector_JST:JST_GH_SM04B-GHS-TB_1x04-1MP_P1.25mm_Horizontal -> RM_Guided_Dart_Base_HW-Footprints:JST_GH_SM04B-GHS-TB_1x04-1MP_P1.25mm_Horizontal
- J5, J6, J7, J8: footprint RWN_Footprints:Connector_Servo_JR_3P_2.54mm_WirePad -> RM_Guided_Dart_Base_HW-Footprints:Connector_Servo_JR_3P_2.54mm_WirePad
- J9: footprint RWN_Footprints:USB-C-TH_KH-TYPE-C-W-16P-T -> RM_Guided_Dart_Base_HW-Footprints:USB-C-TH_KH-TYPE-C-W-16P-T
- L1, L2: footprint Inductor_SMD:L_Changjiang_FTC303020D -> RM_Guided_Dart_Base_HW-Footprints:L_Changjiang_FTC303020D
- L3, L4: footprint Inductor_SMD:L_APV_APH0630 -> RM_Guided_Dart_Base_HW-Footprints:L_APV_APH0630
- Q1, Q2: value AON7544 -> AON7407; footprint Package_SO:Vishay_PowerPAK_1212-8_Single -> RM_Guided_Dart_Base_HW-Footprints:Vishay_PowerPAK_1212-8_Single
- R1, R10, R11, R12, R13, R14, R15, R16, R17, R18, R19, R2, R20, R21, R24, R25, R27, R28, R29, R3, R30, R31, R32, R33, R34, R35, R36, R37, R38, R4, R5, R7, R8, R9: footprint Resistor_SMD:R_0402_1005Metric -> RM_Guided_Dart_Base_HW-Footprints:R_0402_1005Metric
- R22, R23, R26: footprint Resistor_SMD:R_0805_2012Metric -> RM_Guided_Dart_Base_HW-Footprints:R_0805_2012Metric
- R39, R40, R6: footprint Resistor_SMD:R_0603_1608Metric -> RM_Guided_Dart_Base_HW-Footprints:R_0603_1608Metric
- SW1: footprint Button_Switch_SMD:SW_Tactile_SPST_NO_Straight_CK_PTS636Sx25SMTRLFS -> RM_Guided_Dart_Base_HW-Footprints:SW_Tactile_SPST_NO_Straight_CK_PTS636Sx25SMTRLFS
- SW2: footprint Button_Switch_THT:SW_E-Switch_EG1271_SPDT -> RM_Guided_Dart_Base_HW-Footprints:SW_E-Switch_EG1271_SPDT
- U1: footprint RWN_Footprints:LicheeRV_Nano_THT -> RM_Guided_Dart_Base_HW-Footprints:LicheeRV_Nano_THT
- U10, U8, U9: footprint Package_TO_SOT_SMD:SOT-23-5 -> RM_Guided_Dart_Base_HW-Footprints:SOT-23-5
- U11: footprint Package_LGA:Bosch_LGA-16_4.5x3mm_P0.5mm_LayoutBorder7x1y_ClockwisePinNumbering -> RM_Guided_Dart_Base_HW-Footprints:Bosch_LGA-16_4.5x3mm_P0.5mm_LayoutBorder7x1y_ClockwisePinNumbering
- U2: footprint Seeed_Studio_XIAO_Series:XIAO-ESP32-C5-SMD -> RM_Guided_Dart_Base_HW-Footprints:XIAO-ESP32-C5-SMD
- U3, U4: footprint Package_TO_SOT_SMD:TSOT-23-8 -> RM_Guided_Dart_Base_HW-Footprints:TSOT-23-8
- U5: footprint RWN_Footprints:DFN-10-1EP_2x2mm_P0.4mm_EP0.9x1.5mm -> RM_Guided_Dart_Base_HW-Footprints:DFN-10-1EP_2x2mm_P0.4mm_EP0.9x1.5mm
- U6: footprint Package_DFN_QFN:QFN-16-1EP_4x4mm_P0.65mm_EP2.1x2.1mm_ThermalVias -> RM_Guided_Dart_Base_HW-Footprints:QFN-16-1EP_4x4mm_P0.65mm_EP2.1x2.1mm_ThermalVias
- U7: footprint RWN_Footprints:VQFN-14_L3.5-W3.5-P0.50-TL-EP_TPS54620RHLR -> RM_Guided_Dart_Base_HW-Footprints:VQFN-14_L3.5-W3.5-P0.50-TL-EP_TPS54620RHLR
- moved R5 2.75 mm to (154.7, 107.3)
- moved J11 1.05 mm to (102.0, 96.0)
- moved R3 0.06 mm to (108.8, 97.2)
Connections:
- U11 pad 2: unconnected-(U11-NC-Pad2) -> GND
Routing:
- net GND: track 20.1 -> 24.0 mm, vias 77 -> 78
- net /SPI0_SDI: track 38.1 -> 35.2 mm
- net Net-(U2-GPIO9_D9_MISO): track 2.60 -> 4.95 mm
- net /MIPI_RX2_P: track 11.5 -> 10.3 mm
- net /MIPI_RX4_N: track 10.9 -> 9.79 mm
- net /MIPI_RX2_N: track 11.5 -> 10.4 mm
- net /MIPI_RX4_P: track 10.8 -> 9.73 mm
- net /MIPI_RX3_P: track 10.6 -> 9.59 mm
- net /CAM_IO1: track 16.7 -> 15.7 mm
- net +2V8: track 9.18 -> 8.13 mm
- net +1V8: track 30.5 -> 29.4 mm
- net +1V5: track 14.0 -> 13.0 mm
- net /MIPI_RX3_N: track 10.6 -> 9.51 mm
- net /MIPI_RX0_N: track 6.58 -> 5.59 mm
- net /PWM4: track 57.5 -> 58.4 mm
Other:
- board text added: "GND RX"
- board text added: "GND TDI TDO"
- board text added: "IMPOSSIBLE IS NOTHING"
- board text added: "TCK TMS 5V"
- board text added: "TX 5V"

Commit message: V1.2已打板
Parts:
- removed the D6 at (116.0, 84.5)
- added D3: SS54, RM_Guided_Dart_Base_HW-Footprints:D_SMA, B.Cu at (117.9, 82.8)
- added J4: PWM4, RM_Guided_Dart_Base_HW-Footprints:Connector_Servo_JR_3P_2.54mm_WirePad, B.Cu at (137.3, 109.2)
- added R17: 4.7k, RM_Guided_Dart_Base_HW-Footprints:R_0402_1005Metric, B.Cu at (139.7, 88.5)
- added R18: 50k, RM_Guided_Dart_Base_HW-Footprints:R_0402_1005Metric, B.Cu at (138.3, 88.0)
- added R19: 50k, RM_Guided_Dart_Base_HW-Footprints:R_0402_1005Metric, B.Cu at (118.6, 101.0)
- added R44: 10k, RM_Guided_Dart_Base_HW-Footprints:R_0402_1005Metric, B.Cu at (111.6, 88.0)
- J6: value PWM2 -> PWM1
- J7: renamed from J5; value PWM1 -> PWM2
- Q1, Q2: value AON7407 -> AON7403; footprint RM_Guided_Dart_Base_HW-Footprints:Vishay_PowerPAK_1212-8_Single -> Package_SO:Vishay_PowerPAK_1212-8_Single
- R14, R16: value 1k -> 5k
- R30: renamed from R29; value 100k -> 10k
- moved Q1 19.2 mm to (137.5, 90.7), turned to -90 degrees
- moved C14 1.85 mm to (116.4, 100.9), turned to -90 degrees
- moved Q2 1.54 mm to (133.5, 90.3)
- moved R27 1.43 mm to (138.9, 94.0)
- moved C17 1.36 mm to (142.6, 88.7), turned to 90 degrees
- moved C16 1.11 mm to (141.2, 88.7), turned to 90 degrees
- moved R33 1.06 mm to (130.2, 88.6)
- moved C22 1.06 mm to (130.6, 90.6)
- moved C31 0.94 mm to (128.8, 88.2)
- moved R34 0.92 mm to (127.9, 88.2)
- moved R1 0.80 mm to (132.4, 100.9), turned to 90 degrees
- moved R2 0.61 mm to (129.0, 99.1), turned to 90 degrees
- renumbered C14 to C13, C16 to C14, C17 to C15, C13 to C16, C15 to C17, C22 to C21, C23 to C22, C21 to C23, C47 to C30, C30 to C31, C31 to C32, C32 to C33, C33 to C34, C34 to C35, C35 to C36, C36 to C37, C37 to C38, C38 to C39, C39 to C40, C40 to C41, C41 to C42, C42 to C43, C43 to C44, C44 to C45, C45 to C46, C46 to C47, D3 to D4, D4 to D5, D5 to D6, J9 to J10, J10 to J11, J11 to J12, J4 to J5, J7 to J8, J8 to J9, R2 to R1, R1 to R2, R22 to R21, R23 to R22, R17 to R23, R18 to R25, R19 to R26, R21 to R27, R26 to R28, R25 to R29, R27 to R31, R28 to R32, R30 to R33, R31 to R34, R32 to R35, R33 to R36, R34 to R37, R35 to R38, R36 to R39, R37 to R40, R38 to R41, R39 to R42, R40 to R43
Connections:
- C14 pad 2: Net-(U6-CS) -> Net-(U6-VREG)
- C16 pad 1: Net-(U7-VIN) -> Net-(Q1-D)
- C17 pad 1: Net-(U7-VIN) -> Net-(Q1-D)
- J11 pad 1: /Battery/Battery_Power -> GND
- J11 pad 2: GND -> /Battery/Battery_Power
- J2 pad 1: /LCD0_BL+ -> +3V3_SYS_4
- J2 pad 11: unconnected-(J2-Pin_11-Pad11) -> /PWM3
- J2 pad 12: unconnected-(J2-Pin_12-Pad12) -> /PWM4
- J2 pad 14: /SPI0_CS -> Net-(J2-Pin_14)
- J2 pad 15: Net-(J2-Pin_15) -> /SPI0_SDI
- J2 pad 17: /SPI0_SDI -> Net-(J2-Pin_17)
- J2 pad 18: Net-(J2-Pin_18) -> /SPI0_CS
- J2 pad 2: /LCD0_BL+ -> +3V3_SYS_3
- J2 pad 20: /PWM4 -> unconnected-(J2-Pin_20-Pad20)
- J2 pad 21: /PWM3 -> unconnected-(J2-Pin_21-Pad21)
- J2 pad 23: unconnected-(J2-Pin_23-Pad23) -> GND
- J2 pad 24: unconnected-(J2-Pin_24-Pad24) -> /LCD0_BL-
- J2 pad 25: GND -> /LCD0_BL-
- J2 pad 26: +1V8_SYS_1 -> /LCD0_BL-
- J2 pad 27: /LCD0_RESET -> /LCD0_BL-
- J2 pad 28: GND -> unconnected-(J2-Pin_28-Pad28)
- J2 pad 29: +1V8_SYS_2 -> /LCD0_BL+
- J2 pad 3: /LCD0_BL+ -> +1V8_SYS_2
- J2 pad 30: +3V3_SYS_3 -> /LCD0_BL+
- J2 pad 31: +3V3_SYS_4 -> /LCD0_BL+
- J2 pad 4: unconnected-(J2-Pin_4-Pad4) -> GND
- J2 pad 5: /LCD0_BL- -> /LCD0_RESET
- J2 pad 6: /LCD0_BL- -> +1V8_SYS_1
- J2 pad 7: /LCD0_BL- -> GND
- J2 pad 8: /LCD0_BL- -> unconnected-(J2-Pin_8-Pad8)
- J2 pad 9: GND -> unconnected-(J2-Pin_9-Pad9)
- J6 pad 1: /PWM2 -> /PWM1
- J7 pad 1: /PWM1 -> /PWM2
- Q1 pad 5: TypeC_Power -> Net-(Q1-D)
- R1 pad 1: Net-(J2-Pin_18) -> /SPI0_SDO
- R1 pad 2: /SPI0_SDO -> Net-(J2-Pin_14)
- R2 pad 1: Net-(J2-Pin_15) -> /SPI0_SCK
- R2 pad 2: /SPI0_SCK -> Net-(J2-Pin_17)
- R21 pad 1: Net-(D6-K) (its old number) -> TypeC_Power
- R22 pad 2: Net-(D6-K) (its old number) -> TypeC_Power
- R25 pad 2: Net-(U7-VIN) -> Net-(Q1-D)
- SW2 pad 2: Power_IN -> Net-(R17-Pad2)
- SW2 pad 3: Net-(U7-VIN) -> GND
- SW2 pad 5: Power_IN -> Net-(R17-Pad2)
- SW2 pad 6: Net-(U7-VIN) -> GND
- U1 pad 1: /PWM1 -> /PWM2
- U1 pad 2: /PWM2 -> /PWM1
- U6 pad 10: Net-(U6-CS) -> Net-(U6-VREG)
- U6 pad 6: Net-(Q1-G) -> unconnected-(U6-PWR_ON--Pad6)
- U7 pad 4: Net-(U7-VIN) -> Net-(Q1-D)
- U7 pad 5: Net-(U7-VIN) -> Net-(Q1-D)
- U7 pad 6: Net-(U7-VIN) -> Net-(Q1-D)
Routing:
- net Net-(Q1-G): track 30.2 -> 2.74 mm, vias 2 -> 0
- net /PWM2: track 60.0 -> 79.6 mm
- net /PWM1: track 79.6 -> 60.0 mm
- net /UART3_TX: track 74.4 -> 58.5 mm, vias 3 -> 2
- net +5V: track 14.7 -> 27.9 mm
- net Net-(R17-Pad2): track 0.00 -> 8.22 mm
- net Net-(U7-VIN): track 8.20 -> 0.00 mm, vias 6 -> 0
- net Net-(Q1-D): track 0.00 -> 5.92 mm, vias 0 -> 2
- net Net-(U6-VREG): track 0.00 -> 3.75 mm
- net /SPI0_SDO: track 42.0 -> 38.4 mm
- net /PWM3: track 78.1 -> 74.9 mm
- net Net-(J2-Pin_18): track 2.17 -> 0.00 mm
- net Net-(J2-Pin_14): track 0.00 -> 1.94 mm
- net GND: track 24.0 -> 25.6 mm, vias 78 -> 87
- net Net-(Q2-G): track 18.2 -> 16.8 mm
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- added copper zone on B.Cu, net Net-(Q1-D)
- removed copper zone on B.Cu, net Net-(D6-K) (its old number)
- removed copper zone on B.Cu, net Net-(U7-VIN)
- removed copper zone on In2.Cu, net Net-(U7-VIN)
- removed copper zone on In2.Cu, net Power_IN
