File: RM_Guided_Dart_Base_HW.kicad_sch (KiCad schematic)
At the start: 0 parts

Commit message: feat: add camera power schematic, ignore kicad local history
Parts:
- added C1, C2, C3, C6, C7, C9: 1uF, symbol Device:C_Small
- added C4, C5, C8: 22nF, symbol Device:C_Small
- added J1: camera, symbol Connector_Generic_MountingPin:Conn_01x24_MountingPin
- added R1, R2, R3: 10k, symbol Device:R_Small
- added U1: RT9193-18GB, symbol RWN_Symbols:RT9193
- added U2: RT9193-15GB, symbol RWN_Symbols:RT9193
- added U3: RT9193-28GB, symbol RWN_Symbols:RT9193
Connections:
- new net: C2.2, U2.2 (GND)
- new net: C1.2, U1.2 (GND)
- new net: R1.1, U1.3 (EN)
- new net: C4.2, U1.4 (BP)
- new net: R2.1, U2.3 (EN)
- new net: R3.1, U3.3 (EN)
- new net: C5.2, U2.4 (BP)
- new net: C8.2, U3.4 (BP)
- new net: C7.2, U3.2 (GND)
- new net +1V5: C6.2, J1.23 (Pin_23), U2.5 (VOUT)
- new net +1V8: C3.2, J1.22 (Pin_22), U1.5 (VOUT)
- new net +2V8: C9.2, J1.24 (Pin_24), U3.5 (VOUT)
- new net +3V3: C1.1, C2.1, C7.1, R1.2, R2.2, R3.2, U1.1 (VIN), U2.1 (VIN), U3.1 (VIN)
- new net GND: C3.1, C4.1, C5.1, C6.1, C8.1, C9.1, J1.17 (Pin_17), J1.20 (Pin_20), J1.7 (Pin_7), J1.8 (Pin_8), J1.MP (MountPin)
- new net LED-strobe: J1.1 (Pin_1)
- new net MCLK: J1.21 (Pin_21)
- new net MIPI_RCN: J1.18 (Pin_18)
- new net MIPI_RCP: J1.19 (Pin_19)
- new net MIPI_RDN0: J1.9 (Pin_9)
- new net MIPI_RDN1: J1.11 (Pin_11)
- new net MIPI_RDP0: J1.10 (Pin_10)
- new net MIPI_RDP1: J1.12 (Pin_12)
- new net PWDN: J1.3 (Pin_3)
- new net SCL: J1.6 (Pin_6)
- new net SDA: J1.5 (Pin_5)
- new net TRIG: J1.2 (Pin_2)
- no-connect marks 0 -> 5

Commit message: hardware: complete schematic & PCB layout ready for fabrication
Parts:
- removed C1, C2, C3, C6, C7, C9: 1uF, symbol Device:C_Small
- removed C4, C5, C8: 22nF, symbol Device:C_Small
- removed J1: camera, symbol Connector_Generic_MountingPin:Conn_01x24_MountingPin
- removed U1: RT9193-18GB, symbol RWN_Symbols:RT9193
- removed U2: RT9193-15GB, symbol RWN_Symbols:RT9193
- removed U3: RT9193-28GB, symbol RWN_Symbols:RT9193
- added D1: G, LED_SMD:LED_0402_1005Metric, symbol Device:LED
- added H1, H2, H3, H4: MountingHole_Pad, MountingHole:MountingHole_3.2mm_M3_Pad_Via, symbol Mechanical:MountingHole_Pad
- added J1: CSI, RWN_Footprints:FPC-SMD_22P-P1.00_AFC11-S22ICC-00, symbol Connector_Generic_MountingPin:Conn_01x22_MountingPin
- added J2: DSI, Connector_FFC-FPC:Hirose_FH26-31S-0.3SHW_2Rows-31Pins-1MP_P0.60mm_Horizontal, symbol Connector_Generic_MountingPin:Conn_01x31_MountingPin
- added J3: JTAG, Connector_JST:JST_GH_SM06B-GHS-TB_1x06-1MP_P1.25mm_Horizontal, symbol Connector_Generic_MountingPin:Conn_01x06_MountingPin
- added J4: UART3, Connector_JST:JST_GH_SM04B-GHS-TB_1x04-1MP_P1.25mm_Horizontal, symbol Connector_Generic_MountingPin:Conn_01x04_MountingPin
- added J5: PWM1, RWN_Footprints:Connector_Servo_JR_3P_2.54mm_WirePad, symbol Connector_Generic:Conn_01x03
- added J6: PWM2, RWN_Footprints:Connector_Servo_JR_3P_2.54mm_WirePad, symbol Connector_Generic:Conn_01x03
- added J7: PWM3, RWN_Footprints:Connector_Servo_JR_3P_2.54mm_WirePad, symbol Connector_Generic:Conn_01x03
- added J8: PWM4, RWN_Footprints:Connector_Servo_JR_3P_2.54mm_WirePad, symbol Connector_Generic:Conn_01x03
- added R4: 1k, Resistor_SMD:R_0402_1005Metric, symbol Device:R_Small
- added R5, R7: 33R, Resistor_SMD:R_0402_1005Metric, symbol Device:R_Small
- added R6: 33R, Resistor_SMD:R_0603_1608Metric, symbol Device:R_Small
- added SW1: SW_Push, Button_Switch_SMD:SW_Tactile_SPST_NO_Straight_CK_PTS636Sx25SMTRLFS, symbol Switch:SW_Push
- added U1: LicheeRV_Nano, RWN_Footprints:LicheeRV_Nano_THT, symbol Core_moudle:LicheeRV_Nano
- added U2: XIAO-ESP32-C5-DIP, Seeed_Studio_XIAO_Series:XIAO-ESP32-C5-SMD, symbol Seeed_Studio_XIAO_Series:XIAO-ESP32-C5-DIP
- R1, R2, R3: value 10k -> 33R; footprint (none) -> Resistor_SMD:R_0402_1005Metric
Connections:
- net +3V3: now also R4.1; no longer R1.2, R2.2, R3.2
- net GND: now also H1.1, H2.1, H3.1, H4.1, J1.1 (Pin_1), J1.10 (Pin_10), J1.13 (Pin_13), J1.16 (Pin_16), J1.19 (Pin_19), J1.4 (Pin_4), J1.7 (Pin_7), J1.MP (MountPin), J2.10 (Pin_10), J2.13 (Pin_13), J2.19 (Pin_19), J2.22 (Pin_22), J2.25 (Pin_25), J2.28 (Pin_28), J2.9 (Pin_9), J2.MP (MountPin), J3.6 (Pin_6), J3.MP (MountPin), J4.4 (Pin_4), J4.MP (MountPin), J5.3 (Pin_3), J6.3 (Pin_3), J7.3 (Pin_3), J8.3 (Pin_3), SW1.1, U1.26 (GND), U1.3 (GND), U2.13 (GND)
- net at R1.1: now also J2.15 (Pin_15)
- net at R2.1: now also J2.18 (Pin_18)
- net at R3.1: now also J1.14 (Pin_14)
- new net: D1.1 (K), U1.4 (GPIOA_15)
- new net: D1.2 (A), R4.2
- new net: SW1.2, U1.16 (GPIOA_14)
- new net: R7.1, U1.18 (SDIO1_CLK/SPI2_SCK/PWM_9/I2C3_SDA/GPIOP_23)
- new net: R6.1, U1.19 (SDIO1_CMD/SPI2_MOSI/PWM_8/I2C3_SCL/GPIOP_22)
- new net: R5.1, U2.10 (GPIO9_D9_MISO)
- new net +1V8_SYS_1: J2.26 (Pin_26)
- new net +1V8_SYS_2: J2.29 (Pin_29)
- new net +3V3_ESP32-C5: U2.12 (3V3)
- new net +3V3_SYS_1: U1.15 (3V3)
- new net +3V3_SYS_2: J1.22 (Pin_22)
- new net +3V3_SYS_3: J2.30 (Pin_30)
- new net +3V3_SYS_4: J2.31 (Pin_31)
- new net +5V: J3.1 (Pin_1), J4.1 (Pin_1), U1.13 (VSYS), U1.14 (VBUS), U2.14 (VBUS)
- new net +7V2: J5.2 (Pin_2), J6.2 (Pin_2), J7.2 (Pin_2), J8.2 (Pin_2)
- new net CAM_IO0: J1.17 (Pin_17)
- new net CAM_IO1: J1.18 (Pin_18)
- new net CAM_SCL: J1.20 (Pin_20)
- new net CAM_SDA: J1.21 (Pin_21)
- new net CS1_Accel: U1.11 (GPIOA_22/EMMC_CLK/SPI1_SCK)
- new net CS2_Gyro: U1.8 (GPIOA_23/EMMC_CMD/SPI1_MISO)
- new net IMU_SPI2-CS: U1.22 (SDIO1_D3/SPI2_CS/PWM_4/I2C1_SCL/UART3_CTS/GPIOP_18)
- new net IMU_SPI2-MISO: U1.20 (SDIO1_D0/SPI2_MISO/PWM_7/I2C1_SDA/UART3_RTS/GPIOP_21)
- new net IMU_SPI2-MOSI: R6.2
- new net IMU_SPI2-SCK: R7.2
- new net INT1_Accel: U1.7 (GPIOA_24/EMMC_D1/SPI1_CS)
- new net INT2_Accel: U1.10 (GPIOA_25/EMMC_D0/SPI1_MOSI)
- new net INT3_Gyro: U1.12 (GPIOA_26/EMMC_D2)
- new net JTAG_TCK: J3.3 (Pin_3), U1.27 (PWM_6/JTAG_TMS/UART1_RTS/UART1_TX/GPIOA_18)
- new net JTAG_TDI: J3.5 (Pin_5), U1.23 (JTAG_TDI/UART1_TX/UART2_TX/GPIOA_28)
- new net JTAG_TDO: J3.4 (Pin_4), U1.25 (JTAG_TDO/UART1_RX/UART2_RX/GPIOA_29)
- new net JTAG_TMS: J3.2 (Pin_2), U1.28 (PWM_7/JTAG_TCK/UART1_CTS/UART1_RX/GPIOA_19)
- new net LCD0_BL+: J2.1 (Pin_1), J2.2 (Pin_2), J2.3 (Pin_3)
- new net LCD0_BL-: J2.5 (Pin_5), J2.6 (Pin_6), J2.7 (Pin_7), J2.8 (Pin_8)
- new net LCD0_RESET: J2.27 (Pin_27)
- new net MIPI_RX0_N: R3.2
- new net MIPI_RX0_P: J1.15 (Pin_15)
- new net MIPI_RX1_N: J1.11 (Pin_11)
- new net MIPI_RX1_P: J1.12 (Pin_12)
- new net MIPI_RX2_N: J1.8 (Pin_8)
- new net MIPI_RX2_P: J1.9 (Pin_9)
- new net MIPI_RX3_N: J1.5 (Pin_5)
- new net MIPI_RX3_P: J1.6 (Pin_6)
- new net MIPI_RX4_N: J1.2 (Pin_2)
- new net MIPI_RX4_P: J1.3 (Pin_3)
- new net PWM1: J5.1 (Pin_1), U1.1 (GPIOA_17/UART0_RX/PWM_5)
- new net PWM2: J6.1 (Pin_1), U1.2 (GPIOA_16/UART0_TX/PWM_4)
- new net PWM3: J2.21 (Pin_21), J7.1 (Pin_1)
- new net PWM4: J2.20 (Pin_20), J8.1 (Pin_1)
- new net SPI0_CS: J2.14 (Pin_14), U2.1 (GPIO1_A0_D0)
- new net SPI0_HANDSHAKE: U1.9 (GPIOA_27/EMMC_D3), U2.3 (GPIO25_D2)
- new net SPI0_SCK: R1.2, U2.9 (GPIO8_D8_SCK)
- new net SPI0_SDI: J2.17 (Pin_17), R5.2
- new net SPI0_SDO: R2.2, U2.11 (GPIO18_D10_MOSI)
- new net UART3_RX: J4.3 (Pin_3), U1.17 (SDIO1_D1/PWM_6/UART3_RX/GPIOP_20)
- new net UART3_TX: J4.2 (Pin_2), U1.21 (SDIO1_D2/PWM_5/UART3_TX/GPIOP_19)
- new net V_IN: U1.24 (ADC/GPIOB_3)
- no-connect marks 5 -> 15
Other:
- added sheet Battery (Battery.kicad_sch)
- added sheet Camera (Camera.kicad_sch)
- added sheet IMU (IMU.kicad_sch)
- added sheet Power (Power.kicad_sch)
- note added: "PWM[14]"
- note added: "PWM[15]"
- note added: "未使用"

Commit message: hardware: update design and tapeout for fabrication
Parts:
- D1: footprint LED_SMD:LED_0402_1005Metric -> RM_Guided_Dart_Base_HW-Footprints:LED_0402_1005Metric; symbol Device:LED -> RM_Guided_Dart_Base_HW:LED
- H1, H2, H3, H4: footprint MountingHole:MountingHole_3.2mm_M3_Pad_Via -> RM_Guided_Dart_Base_HW-Footprints:MountingHole_3.2mm_M3_Pad_Via; symbol Mechanical:MountingHole_Pad -> RM_Guided_Dart_Base_HW:MountingHole_Pad
- J1: footprint RWN_Footprints:FPC-SMD_22P-P1.00_AFC11-S22ICC-00 -> RM_Guided_Dart_Base_HW-Footprints:FPC-SMD_22P-P1.00_AFC11-S22ICC-00; symbol Connector_Generic_MountingPin:Conn_01x22_MountingPin -> RM_Guided_Dart_Base_HW:Conn_01x22_MountingPin
- J2: footprint Connector_FFC-FPC:Hirose_FH26-31S-0.3SHW_2Rows-31Pins-1MP_P0.60mm_Horizontal -> RM_Guided_Dart_Base_HW-Footprints:Hirose_FH26-31S-0.3SHW_2Rows-31Pins-1MP_P0.60mm_Horizontal; symbol Connector_Generic_MountingPin:Conn_01x31_MountingPin -> RM_Guided_Dart_Base_HW:Conn_01x31_MountingPin
- J3: footprint Connector_JST:JST_GH_SM06B-GHS-TB_1x06-1MP_P1.25mm_Horizontal -> RM_Guided_Dart_Base_HW-Footprints:JST_GH_SM06B-GHS-TB_1x06-1MP_P1.25mm_Horizontal; symbol Connector_Generic_MountingPin:Conn_01x06_MountingPin -> RM_Guided_Dart_Base_HW:Conn_01x06_MountingPin
- J4: footprint Connector_JST:JST_GH_SM04B-GHS-TB_1x04-1MP_P1.25mm_Horizontal -> RM_Guided_Dart_Base_HW-Footprints:JST_GH_SM04B-GHS-TB_1x04-1MP_P1.25mm_Horizontal; symbol Connector_Generic_MountingPin:Conn_01x04_MountingPin -> RM_Guided_Dart_Base_HW:Conn_01x04_MountingPin
- J5, J6, J7, J8: footprint RWN_Footprints:Connector_Servo_JR_3P_2.54mm_WirePad -> RM_Guided_Dart_Base_HW-Footprints:Connector_Servo_JR_3P_2.54mm_WirePad; symbol Connector_Generic:Conn_01x03 -> RM_Guided_Dart_Base_HW:Conn_01x03
- R1, R2, R3, R4, R5, R7: footprint Resistor_SMD:R_0402_1005Metric -> RM_Guided_Dart_Base_HW-Footprints:R_0402_1005Metric; symbol Device:R_Small -> RM_Guided_Dart_Base_HW:R_Small
- R6: footprint Resistor_SMD:R_0603_1608Metric -> RM_Guided_Dart_Base_HW-Footprints:R_0603_1608Metric; symbol Device:R_Small -> RM_Guided_Dart_Base_HW:R_Small
- SW1: footprint Button_Switch_SMD:SW_Tactile_SPST_NO_Straight_CK_PTS636Sx25SMTRLFS -> RM_Guided_Dart_Base_HW-Footprints:SW_Tactile_SPST_NO_Straight_CK_PTS636Sx25SMTRLFS; symbol Switch:SW_Push -> RM_Guided_Dart_Base_HW:SW_Push
- U1: footprint RWN_Footprints:LicheeRV_Nano_THT -> RM_Guided_Dart_Base_HW-Footprints:LicheeRV_Nano_THT; symbol Core_moudle:LicheeRV_Nano -> RM_Guided_Dart_Base_HW:LicheeRV_Nano
- U2: footprint Seeed_Studio_XIAO_Series:XIAO-ESP32-C5-SMD -> RM_Guided_Dart_Base_HW-Footprints:XIAO-ESP32-C5-SMD; symbol Seeed_Studio_XIAO_Series:XIAO-ESP32-C5-DIP -> RM_Guided_Dart_Base_HW:XIAO-ESP32-C5-DIP
Changed lines of the file:
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@@
 	)
 	(symbol
-		(lib_id "Mechanical:MountingHole_Pad")
+		(lib_id "RM_Guided_Dart_Base_HW:MountingHole_Pad")
 		(at 144.78 181.61 0)
 		(unit 1)
@@
 			)
 		)
-		(property "Footprint" "MountingHole:MountingHole_3.2mm_M3_Pad_Via"
+		(property "Footprint" "RM_Guided_Dart_Base_HW-Footprints:MountingHole_3.2mm_M3_Pad_Via"
 			(at 144.78 181.61 0)
 			(hide yes)
@@
 	)
 	(symbol
-		(lib_id "Device:R_Small")
+		(lib_id "RM_Guided_Dart_Base_HW:R_Small")
 		(at 38.1 135.89 90)
 		(unit 1)
@@
 			)
 		)
-		(property "Footprint" "Resistor_SMD:R_0402_1005Metric"
+		(property "Footprint" "RM_Guided_Dart_Base_HW-Footprints:R_0402_1005Metric"
 			(at 38.1 135.89 0)
 			(hide yes)
@@
 	)
 	(symbol
-		(lib_id "Connector_Generic_MountingPin:Conn_01x06_MountingPin")
+		(lib_id "RM_Guided_Dart_Base_HW:Conn_01x06_MountingPin")
 		(at 185.42 137.16 0)
 		(unit 1)
@@
 			)
 		)
-		(property "Footprint" "Connector_JST:JST_GH_SM06B-GHS-TB_1x06-1MP_P1.25mm_Horizontal"
+		(property "Footprint" "RM_Guided_Dart_Base_HW-Footprints:JST_GH_SM06B-GHS-TB_1x06-1MP_P1.25mm_Horizontal"
 			(at 185.42 137.16 0)
 			(hide yes)
@@
 	)
 	(symbol
-		(lib_id "Device:LED")
+		(lib_id "RM_Guided_Dart_Base_HW:LED")
 		(at 78.74 91.44 0)
 		(mirror y)
@@
 			)
 		)
-		(property "Footprint" "LED_SMD:LED_0402_1005Metric"
+		(property "Footprint" "RM_Guided_Dart_Base_HW-Footprints:LED_0402_1005Metric"
 			(at 78.74 91.44 0)
 			(hide yes)
@@
 	)
 	(symbol
-		(lib_id "Mechanical:MountingHole_Pad")
+		(lib_id "RM_Guided_Dart_Base_HW:MountingHole_Pad")
 		(at 74.93 181.61 0)
 		(unit 1)
@@
 			)
 		)
-		(property "Footprint" "MountingHole:MountingHole_3.2mm_M3_Pad_Via"
+		(property "Footprint" "RM_Guided_Dart_Base_HW-Footprints:MountingHole_3.2mm_M3_Pad_Via"
 			(at 74.93 181.61 0)
 			(hide yes)
@@
 	)
 	(symbol
-		(lib_id "Connector_Generic:Conn_01x03")
+		(lib_id "RM_Guided_Dart_Base_HW:Conn_01x03")
 		(at 259.08 132.08 0)
 		(unit 1)
@@
 			)
 		)
-		(property "Footprint" "RWN_Footprints:Connector_Servo_JR_3P_2.54mm_WirePad"
+		(property "Footprint" "RM_Guided_Dart_Base_HW-Footprints:Connector_Servo_JR_3P_2.54mm_WirePad"
 			(at 259.08 132.08 0)
 			(hide yes)
@@
 	)
 	(symbol
-		(lib_id "Device:R_Small")
+		(lib_id "RM_Guided_Dart_Base_HW:R_Small")
 		(at 38.1 143.51 90)
 		(unit 1)
@@
 			)
 		)
-		(property "Footprint" "Resistor_SMD:R_0402_1005Metric"
+		(property "Footprint" "RM_Guided_Dart_Base_HW-Footprints:R_0402_1005Metric"
 			(at 38.1 143.51 0)
 			(hide yes)
@@
 	)
 	(symbol
-		(lib_id "Mechanical:MountingHole_Pad")
+		(lib_id "RM_Guided_Dart_Base_HW:MountingHole_Pad")
 		(at 97.79 181.61 0)
 		(unit 1)
@@
 			)
 		)
-		(property "Footprint" "MountingHole:MountingHole_3.2mm_M3_Pad_Via"
+		(property "Footprint" "RM_Guided_Dart_Base_HW-Footprints:MountingHole_3.2mm_M3_Pad_Via"
 			(at 97.79 181.61 0)
 			(hide yes)
@@
 	)
 	(symbol
-		(lib_id "Switch:SW_Push")
+		(lib_id "RM_Guided_Dart_Base_HW:SW_Push")
 		(at 226.06 114.3 0)
 		(mirror y)
@@
 			)
 		)
-		(property "Footprint" "Button_Switch_SMD:SW_Tactile_SPST_NO_Straight_CK_PTS636Sx25SMTRLFS"
+		(property "Footprint" "RM_Guided_Dart_Base_HW-Footprints:SW_Tactile_SPST_NO_Straight_CK_PTS636Sx25SMTRLFS"
 			(at 226.06 109.22 0)
 			(hide yes)
@@
 	)
 	(symbol
-		(lib_id "Device:R_Small")
+		(lib_id "RM_Guided_Dart_Base_HW:R_Small")
 		(at 54.61 62.23 90)
 		(unit 1)
@@
 			)
 		)
-		(property "Footprint" "Resistor_SMD:R_0402_1005Metric"
+		(property "Footprint" "RM_Guided_Dart_Base_HW-Footprints:R_0402_1005Metric"
 			(at 54.61 62.23 0)
 			(hide yes)
@@
 	)
 	(symbol
-		(lib_id "Connector_Generic_MountingPin:Conn_01x22_MountingPin")
+		(lib_id "RM_Guided_Dart_Base_HW:Conn_01x22_MountingPin")
 		(at 29.21 54.61 0)
 		(mirror y)
@@
 			)
 		)
-		(property "Footprint" "RWN_Footprints:FPC-SMD_22P-P1.00_AFC11-S22ICC-00"
+		(property "Footprint" "RM_Guided_Dart_Base_HW-Footprints:FPC-SMD_22P-P1.00_AFC11-S22ICC-00"
 			(at 29.21 54.61 0)
 			(hide yes)
@@
 	)
 	(symbol
-		(lib_id "Connector_Generic:Conn_01x03")
+		(lib_id "RM_Guided_Dart_Base_HW:Conn_01x03")
 		(at 234.95 132.08 0)
 		(unit 1)
@@
 			)
 		)
-		(property "Footprint" "RWN_Footprints:Connector_Servo_JR_3P_2.54mm_WirePad"
+		(property "Footprint" "RM_Guided_Dart_Base_HW-Footprints:Connector_Servo_JR_3P_2.54mm_WirePad"
 			(at 234.95 132.08 0)
 			(hide yes)
@@
 	)
 	(symbol
-		(lib_id "Device:R_Small")
+		(lib_id "RM_Guided_Dart_Base_HW:R_Small")
 		(at 72.39 91.44 90)
 		(unit 1)
@@
 			)
 		)
-		(property "Footprint" "Resistor_SMD:R_0402_1005Metric"
+		(property "Footprint" "RM_Guided_Dart_Base_HW-Footprints:R_0402_1005Metric"
 			(at 72.39 91.44 0)
 			(hide yes)
@@
 	)
 	(symbol
-		(lib_id "Mechanical:MountingHole_Pad")
+		(lib_id "RM_Guided_Dart_Base_HW:MountingHole_Pad")
 		(at 120.65 181.61 0)
 		(unit 1)
@@
 			)
 		)
-		(property "Footprint" "MountingHole:MountingHole_3.2mm_M3_Pad_Via"
+		(property "Footprint" "RM_Guided_Dart_Base_HW-Footprints:MountingHole_3.2mm_M3_Pad_Via"
 			(at 120.65 181.61 0)
 			(hide yes)
@@
 	)
 	(symbol
-		(lib_id "Connector_Generic_MountingPin:Conn_01x31_MountingPin")
+		(lib_id "RM_Guided_Dart_Base_HW:Conn_01x31_MountingPin")
 		(at 29.21 138.43 0)
 		(mirror y)
@@
 			)
 		)
-		(property "Footprint" "Connector_FFC-FPC:Hirose_FH26-31S-0.3SHW_2Rows-31Pins-1MP_P0.60mm_Horizontal"
+		(property "Footprint" "RM_Guided_Dart_Base_HW-Footprints:Hirose_FH26-31S-0.3SHW_2Rows-31Pins-1MP_P0.60mm_Horizontal"
 			(at 29.21 138.43 0)
 			(hide yes)
@@
 	)
 	(symbol
-		(lib_id "Device:R_Small")
+		(lib_id "RM_Guided_Dart_Base_HW:R_Small")
 		(at 218.44 109.22 90)
 		(unit 1)
@@
 			)
 		)
-		(property "Footprint" "Resistor_SMD:R_0402_1005Metric"
+		(property "Footprint" "RM_Guided_Dart_Base_HW-Footprints:R_0402_1005Metric"
 			(at 218.44 109.22 0)
 			(hide yes)
@@
 	)
 	(symbol
-		(lib_id "Core_moudle:LicheeRV_Nano")
+		(lib_id "RM_Guided_Dart_Base_HW:LicheeRV_Nano")
 		(at 82.55 83.82 0)
 		(unit 1)
@@
 			)
 		)
-		(property "Footprint" "RWN_Footprints:LicheeRV_Nano_THT"
+		(property "Footprint" "RM_Guided_Dart_Base_HW-Footprints:LicheeRV_Nano_THT"
 			(at 95.25 133.35 0)
 			(hide yes)
@@
 	)
 	(symbol
-		(lib_id "Device:R_Small")
+		(lib_id "RM_Guided_Dart_Base_HW:R_Small")
 		(at 139.7 157.48 90)
 		(unit 1)
@@
 			)
 		)
-		(property "Footprint" "Resistor_SMD:R_0402_1005Metric"
+		(property "Footprint" "RM_Guided_Dart_Base_HW-Footprints:R_0402_1005Metric"
 			(at 139.7 157.48 0)
 			(hide yes)
@@
 	)
 	(symbol
-		(lib_id "Connector_Generic:Conn_01x03")
+		(lib_id "RM_Guided_Dart_Base_HW:Conn_01x03")
 		(at 234.95 147.32 0)
 		(unit 1)
@@
 			)
 		)
-		(property "Footprint" "RWN_Footprints:Connector_Servo_JR_3P_2.54mm_WirePad"
+		(property "Footprint" "RM_Guided_Dart_Base_HW-Footprints:Connector_Servo_JR_3P_2.54mm_WirePad"
 			(at 234.95 147.32 0)
 			(hide yes)
@@
 	)
 	(symbol
-		(lib_id "Connector_Generic:Conn_01x03")
+		(lib_id "RM_Guided_Dart_Base_HW:Conn_01x03")
 		(at 259.08 147.32 0)
 		(unit 1)
@@
 			)
 		)
-		(property "Footprint" "RWN_Footprints:Connector_Servo_JR_3P_2.54mm_WirePad"
+		(property "Footprint" "RM_Guided_Dart_Base_HW-Footprints:Connector_Servo_JR_3P_2.54mm_WirePad"
 			(at 259.08 147.32 0)
 			(hide yes)
@@
 	)
 	(symbol
-		(lib_id "Connector_Generic_MountingPin:Conn_01x04_MountingPin")
+		(lib_id "RM_Guided_Dart_Base_HW:Conn_01x04_MountingPin")
 		(at 212.09 137.16 0)
 		(unit 1)
@@
 			)
 		)
-		(property "Footprint" "Connector_JST:JST_GH_SM04B-GHS-TB_1x04-1MP_P1.25mm_Horizontal"
+		(property "Footprint" "RM_Guided_Dart_Base_HW-Footprints:JST_GH_SM04B-GHS-TB_1x04-1MP_P1.25mm_Horizontal"
 			(at 212.09 137.16 0)
 			(hide yes)
@@
 	)
 	(symbol
-		(lib_id "Device:R_Small")
+		(lib_id "RM_Guided_Dart_Base_HW:R_Small")
 		(at 218.44 106.68 90)
 		(unit 1)
@@
 			)
 		)
-		(property "Footprint" "Resistor_SMD:R_0603_1608Metric"
+		(property "Footprint" "RM_Guided_Dart_Base_HW-Footprints:R_0603_1608Metric"
 			(at 218.44 106.68 0)
 			(hide yes)
@@
 	)
 	(symbol
-		(lib_id "Seeed_Studio_XIAO_Series:XIAO-ESP32-C5-DIP")
+		(lib_id "RM_Guided_Dart_Base_HW:XIAO-ESP32-C5-DIP")
 		(at 109.22 160.02 0)
 		(unit 1)
@@
 			)
 		)
-		(property "Footprint" "Seeed_Studio_XIAO_Series:XIAO-ESP32-C5-SMD"
+		(property "Footprint" "RM_Guided_Dart_Base_HW-Footprints:XIAO-ESP32-C5-SMD"
 			(at 100.33 154.94 0)
 			(hide yes)

Commit message: V1.2已打板
Parts:
- added J4: PWM4, RM_Guided_Dart_Base_HW-Footprints:Connector_Servo_JR_3P_2.54mm_WirePad, symbol RM_Guided_Dart_Base_HW:Conn_01x03
- J6: value PWM2 -> PWM1
- J7: renamed from J5; value PWM1 -> PWM2
- renumbered J4 to J5, J7 to J8, J8 to J9, R2 to R1, R1 to R2
Connections:
- net +1V8_SYS_1: now also J2.6 (Pin_6); no longer J2.26 (Pin_26)
- net +1V8_SYS_2: now also J2.3 (Pin_3); no longer J2.29 (Pin_29)
- net +3V3_SYS_3: now also J2.2 (Pin_2); no longer J2.30 (Pin_30)
- net +3V3_SYS_4: now also J2.1 (Pin_1); no longer J2.31 (Pin_31)
- net +5V: now also J4.2 (Pin_2)
- net GND: now also J2.23 (Pin_23), J2.4 (Pin_4), J2.7 (Pin_7), J4.1 (Pin_1); no longer J2.25 (Pin_25), J2.28 (Pin_28), J2.9 (Pin_9)
- net LCD0_BL+: now also J2.29 (Pin_29), J2.30 (Pin_30), J2.31 (Pin_31); no longer J2.1 (Pin_1), J2.2 (Pin_2), J2.3 (Pin_3)
- net LCD0_BL-: now also J2.24 (Pin_24), J2.25 (Pin_25), J2.26 (Pin_26), J2.27 (Pin_27); no longer J2.5 (Pin_5), J2.6 (Pin_6), J2.7 (Pin_7), J2.8 (Pin_8)
- net LCD0_RESET: now also J2.5 (Pin_5); no longer J2.27 (Pin_27)
- net PWM1: now also J6.1 (Pin_1), U1.2 (GPIOA_16/UART0_TX/PWM_4); no longer J7.1 (Pin_1), U1.1 (GPIOA_17/UART0_RX/PWM_5)
- net PWM2: now also J7.1 (Pin_1), U1.1 (GPIOA_17/UART0_RX/PWM_5); no longer J6.1 (Pin_1), U1.2 (GPIOA_16/UART0_TX/PWM_4)
- net PWM3: now also J2.11 (Pin_11); no longer J2.21 (Pin_21)
- net PWM4: now also J2.12 (Pin_12); no longer J2.20 (Pin_20)
- net SPI0_CS: now also J2.18 (Pin_18); no longer J2.14 (Pin_14)
- net SPI0_SCK: now also R2.1; no longer R2.2
- net SPI0_SDI: now also J2.15 (Pin_15); no longer J2.17 (Pin_17)
- net SPI0_SDO: now also R1.1; no longer R1.2
- new net: J2.17 (Pin_17), R2.2
- new net: J2.14 (Pin_14), R1.2
- new net UART: J4.3 (Pin_3)
Other:
- note added: "AON7407 Vgs耐压只有+-8V"
- note added: "DSI排线座反了"
- note added: "IMU加热电阻最好加上"
- note added: "XT30接口正负颠倒"
- note added: "充电回路加了typec输入mos后 在开关切换瞬间会烧tp5100"
- note added: "双通道开关瞬间会有大电流，直接上电反而不会， 同时TP5100会瞬间烧穿，目前未排查出原因"
- note added: "取消丝印反显"
- note added: "已解决"
- note added: "无需解决"
- note added: "最好用mos作开关"
- note added: "错误："
- note added: "镖头灯未加"
- moved on the sheet: J5, J6, J7, R1, R2
